File: AWG.kicad_pcb (KiCad board)
At the start: 2 copper layers, 140 x 75 mm, 81 parts, among them J1001 Conn_01x03, J1002 Conn_01x05, J1003 Conn_01x06, J1005 Conn_01x01, J1006 Conn_01x01, J1007 Conn_01x01, J1008 Conn_01x01, J1009 Conn_01x01, J1010 Conn_01x01, J1011 Conn_01x01, J1012 Conn_01x01, J1013 Conn_01x05, J2 Conn afficheur, J5 SMA, Q1001 NTE2633, Q1002 NTE2634, U1 Pico, U1001 L7812, U1002 L7912, U1003 L7805, U1004 L7905, U3 AD8055ARZ

Commit message: Redesign
Parts:
- removed C1001, C1002, C1005, C1006, C1009, C1010: 100u 50V, Capacitor_THT:CP_Radial_D10.0mm_P2.50mm_P5.00mm
- removed C1003, C1004, C1007, C1008, C1011, C1012, C1013, C1015, C1017: 100n, Capacitor_SMD:C_0805_2012Metric_Pad1.18x1.45mm_HandSolder
- removed HS1001, HS1002: Heatsink, Heatsink:Heatsink_Aavid-TV5G_TO220_Horizontal
- removed J1001: Conn_01x03, Connector_Molex:Molex_KK-254_AE-6410-03A_1x03_P2.54mm_Vertical
- removed J1002, J1013: Conn_01x05, Connector_Molex:Molex_KK-254_AE-6410-05A_1x05_P2.54mm_Vertical
- removed J1009, J1010, J1011, J1012: Conn_01x01, MountingHole:MountingHole_3.2mm_M3_Pad_Via
- removed the J2 at (225.0, 95.0)
- removed Q1001: NTE2633, Package_TO_SOT_THT:TO-220-3_Horizontal_TabDown
- removed Q1002: NTE2634, Package_TO_SOT_THT:TO-220-3_Horizontal_TabDown
- removed R1001, R1002, R1003, R1004, R1005: 1k, Resistor_SMD:R_0603_1608Metric_Pad0.98x0.95mm_HandSolder
- removed the R26 at (179.4, 81.6)
- removed the R30 at (167.5, 87.5)
- removed RV1: 100R, Potentiometer_THT:Potentiometer_Piher_PT-10-V10_Vertical_Hole
- removed U1001: L7812, Package_TO_SOT_SMD:TO-252-2
- removed U1002: L7912, Package_TO_SOT_SMD:TO-252-2
- removed U1003: L7805, Package_TO_SOT_SMD:TO-252-2
- removed U1004: L7905, Package_TO_SOT_SMD:TO-252-2
- added C1: 22u, Capacitor_SMD:C_1210_3225Metric, F.Cu at (262.0, 64.0)
- added C10: 22u, Capacitor_SMD:C_1210_3225Metric, F.Cu at (177.8, 76.0)
- added C11: 22u, Capacitor_SMD:C_1210_3225Metric, F.Cu at (207.7, 67.6)
- added C12: 22u, Capacitor_SMD:C_1210_3225Metric, F.Cu at (211.1, 67.6)
- added C13: 100n, Capacitor_SMD:C_0603_1608Metric, F.Cu at (178.0, 83.0)
- added C14: 100n, Capacitor_SMD:C_0603_1608Metric, F.Cu at (188.4, 84.2)
- added C15: 22u, Capacitor_SMD:C_1210_3225Metric, F.Cu at (217.5, 85.0)
- added C16: 22u, Capacitor_SMD:C_1210_3225Metric, F.Cu at (270.5, 85.5)
- added C17: 100n, Capacitor_SMD:C_0603_1608Metric, F.Cu at (218.0, 87.5)
- added C18: DNP, Capacitor_SMD:C_0603_1608Metric, F.Cu at (192.8, 89.4)
- added C19: DNP, Capacitor_SMD:C_0603_1608Metric, F.Cu at (228.1, 93.0)
- added C2: 22u, Capacitor_SMD:C_1210_3225Metric, F.Cu at (216.7, 63.4)
- added C20: 100n, Capacitor_SMD:C_0603_1608Metric, F.Cu at (186.4, 93.2)
- added C21: 100n, Capacitor_SMD:C_0603_1608Metric, F.Cu at (233.0, 93.5)
- added C22: 100n, Capacitor_SMD:C_0603_1608Metric, F.Cu at (212.0, 93.8)
- added C23: 100n, Capacitor_SMD:C_0603_1608Metric, F.Cu at (224.0, 94.4)
- added C24: 22u, Capacitor_SMD:C_1210_3225Metric, F.Cu at (209.5, 94.5)
- added C25: 100n, Capacitor_SMD:C_0603_1608Metric, F.Cu at (267.0, 95.5)
- added C26: 100n, Capacitor_SMD:C_0603_1608Metric, F.Cu at (175.8, 96.0)
- added C27: 22u, Capacitor_SMD:C_1210_3225Metric, F.Cu at (181.0, 101.5)
- added C28: 22u, Capacitor_SMD:C_1210_3225Metric, F.Cu at (271.6, 102.3)
- added C29: 100u, Capacitor_SMD:CP_Elec_6.3x5.4_Nichicon, F.Cu at (175.5, 104.0)
- added C8: 22u, Capacitor_SMD:C_1210_3225Metric, F.Cu at (223.7, 67.9)
- added D3: 1N4148WS, Diode_SMD:D_SOD-323, F.Cu at (188.6, 80.6)
- added D4: 1N5819WS, Diode_SMD:D_SOD-323, F.Cu at (267.2, 89.0)
- added D5: 1N4148WS, Diode_SMD:D_SOD-323, F.Cu at (186.6, 96.6)
- added H1: MountingHole, MountingHole:MountingHole_3.2mm_M3, F.Cu at (194.1, 64.8)
- added H2: MountingHole, MountingHole:MountingHole_3.2mm_M3, F.Cu at (155.0, 65.0)
- added H3: MountingHole, MountingHole:MountingHole_3.2mm_M3, F.Cu at (178.0, 65.0)
- added H4: MountingHole, MountingHole:MountingHole_3.2mm_M3, F.Cu at (194.1, 108.8)
- added H5: MountingHole, MountingHole:MountingHole_3.2mm_M3, F.Cu at (197.5, 129.0)
- added H6: MountingHole, MountingHole:MountingHole_3.2mm_M3, F.Cu at (197.0, 151.5)
- added J3: Conn_01x03, Connector_JST:JST_XH_S3B-XH-A_1x03_P2.50mm_Horizontal, F.Cu at (267.0, 59.0)
- added J4: BNC, Connector_Coaxial:BNC_TEConnectivity_1478035_Horizontal, F.Cu at (148.0, 87.5)
- added J9: Controls, Connector_PinSocket_2.54mm:PinSocket_1x06_P2.54mm_Vertical, B.Cu at (142.5, 136.0)
- added L1: 68u, Inductor_SMD:L_Wuerth_MAPI-3020, F.Cu at (203.9, 72.4)
- added L2: 68u, Inductor_SMD:L_Wuerth_MAPI-3020, F.Cu at (182.0, 76.5)
- added L3: 68u, Inductor_SMD:L_Wuerth_MAPI-3020, F.Cu at (208.1, 72.0)
- added L4: 68u, Inductor_SMD:L_Wuerth_MAPI-3020, F.Cu at (216.5, 72.7)
- added L5: 68u, Inductor_SMD:L_Wuerth_MAPI-3020, F.Cu at (221.0, 72.5)
- added L6: 51n, Inductor_THT:L_Axial_L7.0mm_D3.3mm_P10.16mm_Horizontal_Fastron_MICC, F.Cu at (205.5, 88.6)
- added L7: 68u, Inductor_SMD:L_Wuerth_MAPI-3020, F.Cu at (270.5, 89.5)
- added L8: 68u, Inductor_SMD:L_Wuerth_MAPI-3020, F.Cu at (185.0, 101.0)
- added L9: 68u, Inductor_SMD:L_Wuerth_MAPI-3020, F.Cu at (267.5, 104.0)
- added Q1: FZT653, Package_TO_SOT_SMD:SOT-223-3_TabPin2, F.Cu at (183.1, 82.1)
- added Q2: S9015, Package_TO_SOT_SMD:SOT-23, F.Cu at (270.5, 93.5)
- added Q3: FZT753, Package_TO_SOT_SMD:SOT-223-3_TabPin2, F.Cu at (181.1, 95.2)
- added R17: 27, Resistor_SMD:R_0603_1608Metric, F.Cu at (271.0, 79.0)
- added R18: 27, Resistor_SMD:R_0603_1608Metric, F.Cu at (270.9, 81.0)
- added R19: 27, Resistor_SMD:R_0603_1608Metric, F.Cu at (270.9, 82.6)
- added R20: 1k, Resistor_SMD:R_0603_1608Metric, F.Cu at (190.0, 84.1)
- added R35: 1k, Resistor_SMD:R_0603_1608Metric, F.Cu at (222.2, 91.0)
- added R36: DNP, Resistor_SMD:R_0603_1608Metric, F.Cu at (226.6, 93.0)
- added R37: 1k, Resistor_SMD:R_0603_1608Metric, F.Cu at (188.0, 93.2)
- added R38: 1k, Resistor_SMD:R_0603_1608Metric, F.Cu at (215.5, 94.5)
- added R39: 1k, Resistor_SMD:R_0603_1608Metric, F.Cu at (219.0, 94.5)
- added R40: 1k, Resistor_SMD:R_0603_1608Metric, F.Cu at (221.5, 94.5)
- added R41: 68k, Resistor_SMD:R_0603_1608Metric, F.Cu at (232.9, 95.0)
- added R42: 68k, Resistor_SMD:R_0603_1608Metric, F.Cu at (224.0, 96.0)
- added R43: 2k, Resistor_SMD:R_0603_1608Metric, F.Cu at (270.4, 96.5)
- added R5: 68k, Resistor_SMD:R_0603_1608Metric, F.Cu at (200.9, 69.4)
- added R6: 12k, Resistor_SMD:R_0603_1608Metric, F.Cu at (213.6, 70.6)
- added R7: 68k, Resistor_SMD:R_0603_1608Metric, F.Cu at (213.6, 73.6)
- added R8: 12k, Resistor_SMD:R_0603_1608Metric, F.Cu at (200.9, 72.4)
- added SW1: Prev, Module:Square_PB, F.Cu at (155.0, 142.0)
- added SW2: Next, Module:Square_PB, F.Cu at (195.0, 142.0)
- added SW3: Encoder, Rotary_Encoder:RotaryEncoder_Alps_EC12E-Switch_Vertical_H20mm, F.Cu at (172.5, 149.8)
- added TP1: TestPoint_2Pole, Module:TestPoint_2Pads_Pitch2.54mm_Drill1mm, F.Cu at (167.0, 77.2)
- added TP2: TestPoint_2Pole, Module:TestPoint_2Pads_Pitch2.54mm_Drill1mm, F.Cu at (222.0, 85.2)
- added TP3: TestPoint_2Pole, Module:TestPoint_2Pads_Pitch2.54mm_Drill1mm, F.Cu at (190.0, 88.5)
- added TP4: TestPoint_2Pole, Module:TestPoint_2Pads_Pitch2.54mm_Drill1mm, F.Cu at (208.4, 88.5)
- added TP5: TestPoint_2Pole, Module:TestPoint_2Pads_Pitch2.54mm_Drill1mm, F.Cu at (224.4, 91.2)
- added TP6: TestPoint_2Pole, Module:TestPoint_2Pads_Pitch2.54mm_Drill1mm, F.Cu at (205.5, 94.2)
- added TP7: TestPoint_2Pole, Module:TestPoint_2Pads_Pitch2.54mm_Drill1mm, F.Cu at (169.5, 100.5)
- added U2: BD9G101G, Package_TO_SOT_SMD:SOT-23-6, F.Cu at (203.9, 66.4)
- added U4: LMH6658, Package_SO:SOIC-8_3.9x4.9mm_P1.27mm, F.Cu at (216.5, 91.0)
- C3: value 100n -> 22u; footprint Capacitor_SMD:C_0805_2012Metric_Pad1.18x1.45mm_HandSolder -> Capacitor_SMD:C_1210_3225Metric
- C4: footprint Capacitor_SMD:C_0805_2012Metric_Pad1.18x1.45mm_HandSolder -> Capacitor_SMD:C_0603_1608Metric; moved to F.Cu
- C5: value 100n -> 100u; footprint Capacitor_SMD:C_0805_2012Metric_Pad1.18x1.45mm_HandSolder -> Capacitor_SMD:CP_Elec_6.3x5.4_Nichicon; moved to F.Cu
- C6: value 1mF -> 22u; footprint Capacitor_SMD:C_1812_4532Metric_Pad1.57x3.40mm_HandSolder -> Capacitor_SMD:C_1210_3225Metric
- C7: value 3.3p -> 22u; footprint Capacitor_SMD:C_0805_2012Metric_Pad1.18x1.45mm_HandSolder -> Capacitor_SMD:C_1210_3225Metric
- C9: footprint Capacitor_SMD:C_0805_2012Metric_Pad1.18x1.45mm_HandSolder -> Capacitor_SMD:C_0603_1608Metric
- D1, D2: value 4148 -> 1N5819WS; footprint Diode_SMD:D_MicroMELF_Handsoldering -> Diode_SMD:D_SOD-323
- J5: value SMA -> Conn_01x14; footprint SMA_PINS:SMA_EDGE_NRW -> Connector_PinSocket_2.54mm:PinSocket_1x14_P2.54mm_Vertical; moved to F.Cu
- J6: renamed from J1003; value Conn_01x06 -> Controls; footprint Connector_Molex:Molex_KK-254_AE-6410-06A_1x06_P2.54mm_Vertical -> Connector_PinHeader_2.54mm:PinHeader_1x06_P2.54mm_Vertical
- R1: renamed from R25; footprint Resistor_SMD:R_0603_1608Metric_Pad0.98x0.95mm_HandSolder -> Resistor_SMD:R_0603_1608Metric
- R10: renamed from R11; footprint Resistor_SMD:R_0603_1608Metric_Pad0.98x0.95mm_HandSolder -> Resistor_SMD:R_0603_1608Metric
- R11: renamed from R22; footprint Resistor_SMD:R_0603_1608Metric_Pad0.98x0.95mm_HandSolder -> Resistor_SMD:R_0603_1608Metric
- R12: renamed from R10; footprint Resistor_SMD:R_0603_1608Metric_Pad0.98x0.95mm_HandSolder -> Resistor_SMD:R_0603_1608Metric
- R13: renamed from R21; footprint Resistor_SMD:R_0603_1608Metric_Pad0.98x0.95mm_HandSolder -> Resistor_SMD:R_0603_1608Metric
- R14: renamed from R9; footprint Resistor_SMD:R_0603_1608Metric_Pad0.98x0.95mm_HandSolder -> Resistor_SMD:R_0603_1608Metric
- R15: renamed from R20; footprint Resistor_SMD:R_0603_1608Metric_Pad0.98x0.95mm_HandSolder -> Resistor_SMD:R_0603_1608Metric
- R16: renamed from R8; footprint Resistor_SMD:R_0603_1608Metric_Pad0.98x0.95mm_HandSolder -> Resistor_SMD:R_0603_1608Metric
- R2: renamed from R13; footprint Resistor_SMD:R_0603_1608Metric_Pad0.98x0.95mm_HandSolder -> Resistor_SMD:R_0603_1608Metric
- R21: renamed from R19; footprint Resistor_SMD:R_0603_1608Metric_Pad0.98x0.95mm_HandSolder -> Resistor_SMD:R_0603_1608Metric
- R22: renamed from R7; footprint Resistor_SMD:R_0603_1608Metric_Pad0.98x0.95mm_HandSolder -> Resistor_SMD:R_0603_1608Metric
- R23: renamed from R18; footprint Resistor_SMD:R_0603_1608Metric_Pad0.98x0.95mm_HandSolder -> Resistor_SMD:R_0603_1608Metric
- R24: renamed from R6; footprint Resistor_SMD:R_0603_1608Metric_Pad0.98x0.95mm_HandSolder -> Resistor_SMD:R_0603_1608Metric
- R25: renamed from R17; footprint Resistor_SMD:R_0603_1608Metric_Pad0.98x0.95mm_HandSolder -> Resistor_SMD:R_0603_1608Metric
- R26: renamed from R5; footprint Resistor_SMD:R_0603_1608Metric_Pad0.98x0.95mm_HandSolder -> Resistor_SMD:R_0603_1608Metric
- R27: value 680R -> 1; footprint Resistor_SMD:R_0603_1608Metric_Pad0.98x0.95mm_HandSolder -> Resistor_SMD:R_1206_3216Metric
- R28: value 680R -> 10; footprint Resistor_SMD:R_0603_1608Metric_Pad0.98x0.95mm_HandSolder -> Resistor_SMD:R_0603_1608Metric; moved to F.Cu
- R29: renamed from R16; footprint Resistor_SMD:R_0603_1608Metric_Pad0.98x0.95mm_HandSolder -> Resistor_SMD:R_0603_1608Metric
- R3: renamed from R24; footprint Resistor_SMD:R_0603_1608Metric_Pad0.98x0.95mm_HandSolder -> Resistor_SMD:R_0603_1608Metric
- R30: renamed from R4; footprint Resistor_SMD:R_0603_1608Metric_Pad0.98x0.95mm_HandSolder -> Resistor_SMD:R_0603_1608Metric
- R31: value 1k -> 1; footprint Resistor_SMD:R_0603_1608Metric_Pad0.98x0.95mm_HandSolder -> Resistor_SMD:R_1206_3216Metric
- R32: footprint Resistor_SMD:R_0603_1608Metric_Pad0.98x0.95mm_HandSolder -> Resistor_SMD:R_0603_1608Metric
- R33: value 3R3 -> 0; footprint Resistor_SMD:R_1210_3225Metric_Pad1.30x2.65mm_HandSolder -> Resistor_SMD:R_0603_1608Metric; moved to F.Cu
- R34: value 3R3 -> 1k; footprint Resistor_SMD:R_1210_3225Metric_Pad1.30x2.65mm_HandSolder -> Resistor_SMD:R_0603_1608Metric; moved to F.Cu
- R4: renamed from R12; footprint Resistor_SMD:R_0603_1608Metric_Pad0.98x0.95mm_HandSolder -> Resistor_SMD:R_0603_1608Metric
- R9: renamed from R23; footprint Resistor_SMD:R_0603_1608Metric_Pad0.98x0.95mm_HandSolder -> Resistor_SMD:R_0603_1608Metric
- U1: value Pico -> BD9G101G; footprint Pi_Pico:RPi_Pico_SMD_TH -> Package_TO_SOT_SMD:SOT-23-6
- U3: value AD8055ARZ -> Pico; footprint Package_SO:SO-8_3.9x4.9mm_P1.27mm -> MCU_RaspberryPi_and_Boards:RPi_Pico_SMD
- moved J5 134.0 mm to (275.1, 103.3)
- moved U3 73.8 mm to (246.4, 87.1), turned to 0 degrees
- moved R33 59.9 mm to (227.6, 90.5), turned to 180 degrees
- moved C3 47.9 mm to (262.0, 69.5)
- moved R34 46.7 mm to (208.6, 91.0), turned to 180 degrees
- moved C7 45.6 mm to (220.4, 67.9)
- moved D2 45.1 mm to (216.4, 69.6), turned to 0 degrees
- moved R32 42.4 mm to (211.0, 90.0), turned to 90 degrees
- moved R9 42.0 mm to (227.5, 72.0), turned to 180 degrees
- moved R21 41.5 mm to (227.6, 84.5), turned to 180 degrees
- moved R11 41.5 mm to (227.5, 73.5), turned to 180 degrees
- moved R23 41.2 mm to (227.6, 86.0), turned to 180 degrees
- moved R13 41.1 mm to (227.5, 75.0), turned to 180 degrees
- moved R25 41.0 mm to (227.6, 87.5), turned to 180 degrees
- moved R15 40.9 mm to (227.5, 76.5), turned to 180 degrees
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- renumbered J1006 to J1, J1007 to J2, J1008 to J7, J1005 to J8
Connections:
- C3 pad 1: +5V -> GND
- C3 pad 2: GND -> +3V3
- C4 pad 1: +3V3 -> Net-(C4-Pad1)
- C4 pad 2: GND -> Net-(C4-Pad2)
- C5 pad 1: +5V -> +12V
- C6 pad 1: Net-(C6-Pad1) -> /power/-12V_UNFIL
- C6 pad 2: Net-(C6-Pad2) -> GND
- C7 pad 1: Net-(C6-Pad1) -> GND
- C7 pad 2: GND -> +5VD
- C9 pad 1: GND -> Net-(C9-Pad1)
- C9 pad 2: -5V -> Net-(C9-Pad2)
- D1 pad 1: Net-(D1-Pad1) -> Net-(C4-Pad1)
- D1 pad 2: Net-(D1-Pad2) -> /power/-12V_UNFIL
- D2 pad 1: Net-(D2-Pad1) -> Net-(C9-Pad1)
- D2 pad 2: Net-(D2-Pad2) -> GND
- J5 pad 1: Net-(J5-Pad1) -> /LCD_3V3
- J6 pad 1: Net-(C1011-Pad1) -> /ENC_A
- J6 pad 2: Net-(C1012-Pad1) -> /ENC_B
- J6 pad 3: Net-(C1013-Pad1) -> /ENC_SW
- J6 pad 4: Net-(C1015-Pad1) -> /B_NE
- J6 pad 5: Net-(C1017-Pad1) -> /B_PR
- R10 pad 1: Net-(R11-Pad1) -> Net-(R10-Pad1)
- R12 pad 1: Net-(R10-Pad1) -> Net-(R12-Pad1)
- R14 pad 1: Net-(R9-Pad1) -> Net-(R14-Pad1)
- R16 pad 1: Net-(R8-Pad1) -> Net-(R16-Pad1)
- R2 pad 1: Net-(R13-Pad1) -> Net-(R2-Pad1)
- R22 pad 1: Net-(R7-Pad1) -> Net-(R22-Pad1)
- R24 pad 1: Net-(R6-Pad1) -> Net-(R24-Pad1)
- R26 pad 1: Net-(R5-Pad1) -> Net-(R26-Pad1)
- R27 pad 1: Net-(R27-Pad1) -> Net-(Q1-Pad3)
- R27 pad 2: GND -> /amp/OUT
- R28 pad 1: Net-(R27-Pad1) -> Net-(L6-Pad1)
- R29 pad 1: Net-(C6-Pad2) -> /amp/IN
- R30 pad 1: Net-(R4-Pad1) -> Net-(R30-Pad1)
- R30 pad 2: Net-(C6-Pad2) -> /amp/IN
- R31 pad 1: +12V -> /amp/OUT
- R31 pad 2: Net-(D1-Pad2) -> Net-(R31-Pad2)
- R32 pad 1: Net-(D2-Pad1) -> Net-(R32-Pad1)
- R32 pad 2: -12V -> Net-(L6-Pad1)
- R33 pad 1: Net-(Q1001-Pad1) -> /amp/IN
- R33 pad 2: Net-(J5-Pad1) -> Net-(C19-Pad1)
- R34 pad 1: Net-(J5-Pad1) -> Net-(R32-Pad1)
- R34 pad 2: Net-(Q1002-Pad1) -> GND
- R4 pad 1: Net-(R12-Pad1) -> Net-(R4-Pad1)
- U1 pad 1: Net-(R13-Pad1) -> Net-(C9-Pad2)
- U1 pad 2: Net-(R12-Pad1) -> GND
- U1 pad 3: GND -> Net-(R7-Pad1)
- U1 pad 4: Net-(R11-Pad1) -> /power/+12V_UNFIL
- U1 pad 5: Net-(R10-Pad1) -> /power/+12V_UNFIL
- U1 pad 6: Net-(R9-Pad1) -> Net-(C9-Pad1)
- U3 pad 1: unconnected-(U3-Pad1) -> Net-(R2-Pad1)
- U3 pad 2: Net-(R27-Pad1) -> Net-(R4-Pad1)
- U3 pad 3: Net-(C6-Pad1) -> GND
- U3 pad 4: -5V -> Net-(R10-Pad1)
- U3 pad 5: unconnected-(U3-Pad5) -> Net-(R12-Pad1)
- U3 pad 6: Net-(R28-Pad2) -> Net-(R14-Pad1)
- U3 pad 7: +5V -> Net-(R16-Pad1)
- U3 pad 8: unconnected-(U3-Pad8) -> GND
Routing:
- net +5V: track 246.0 -> 40.0 mm
- net -12V: track 220.7 -> 34.4 mm, vias 0 -> 6
- net /B_NE: track 0.00 -> 185.1 mm, vias 0 -> 1
- net +12V: track 214.4 -> 35.3 mm, vias 0 -> 7
- net /ENC_A: track 0.00 -> 171.0 mm, vias 0 -> 2
- net /ENC_B: track 0.00 -> 158.9 mm, vias 0 -> 2
- net /power/-12V_UNFIL: track 0.00 -> 152.2 mm, vias 0 -> 17
- net /B_PR: track 0.00 -> 140.9 mm, vias 0 -> 2
- net /ENC_SW: track 0.00 -> 138.3 mm, vias 0 -> 2
- net -5V: track 187.7 -> 55.0 mm, vias 0 -> 5
- net /power/+12V_UNFIL: track 0.00 -> 117.4 mm, vias 0 -> 3
- net +5VD: track 0.00 -> 68.9 mm, vias 0 -> 3
- net Net-(J5-Pad1): track 61.6 -> 0.00 mm
- net +3V3: track 89.2 -> 45.6 mm, vias 0 -> 4
- net /amp/OUT: track 0.00 -> 37.8 mm
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- added copper zone on B.Cu, net +12V
- added copper zone on F.Cu, net +12V
- added copper zone on B.Cu, net -12V
- added copper zone on F.Cu, net /power/-12V_UNFIL
- added copper zone on In1.Cu, net /power/-12V_UNFIL
- added copper zone on In1.Cu, net GND
- added copper zone on In2.Cu, net GND
- added copper zone on F.Cu, net Net-(C4-Pad1)
- added copper zone on F.Cu, net Net-(C9-Pad1)
- added copper zone on F.Cu, net Net-(D4-Pad1)
Other:
- board size 140 x 75 mm -> 140 x 108.5 mm
- copper layers 2 -> 4
- board text added: "+12"
- board text added: "-12"
- board text added: "Controls"
- board text added: "flaviutamas.com/p/awg-15M"
- board text removed: "+12V +5V GND -5V -12V"
- board text removed: "+15V -15V Power In"
- board text removed: "+5V MISO CS Gnd SCK MOSI D/C Reset Led On Rst Raspi"
- board text removed: "Output"
- board text removed: "To Frontpanel"
