File: AWG.kicad_sch (KiCad schematic)
At the start: 92 parts, among them J1001 Conn_01x03, J1002 Conn_01x05, J1003 Conn_01x06, J1004 Conn_01x06, J1005 Conn_01x01, J1006 Conn_01x01, J1007 Conn_01x01, J1008 Conn_01x01, J1009 Conn_01x01, J1010 Conn_01x01, J1011 Conn_01x01, J1012 Conn_01x01, J1013 Conn_01x05, J2 Conn afficheur, J5 SMA, J6 SMA, J7 BNC, Q1001 NTE2633, Q1002 NTE2634, SW1 Reset, SW2 Encodeur sur façade, SW3 Next, SW4 Previous, SW5 AC/DC, SW6 50R/Low Z, U1 Pico, U1001 L7812, U1002 L7912, U1003 L7805, U1004 L7905, U3 AD8055ARZ

Commit message: Redesign
Parts:
- removed C1001, C1002, C1005, C1006, C1009, C1010: 100u 50V, Capacitor_THT:CP_Radial_D10.0mm_P2.50mm_P5.00mm, symbol Device:CP_Small
- removed C1003, C1004, C1007, C1008, C1011, C1012, C1013, C1015, C1017, C4, C5, C9: 100n, Capacitor_SMD:C_0805_2012Metric_Pad1.18x1.45mm_HandSolder, symbol Device:C_Small
- removed C13: 1mf, symbol Device:C_Small
- removed C6: 1mF, Capacitor_SMD:C_1812_4532Metric_Pad1.57x3.40mm_HandSolder, symbol Device:C_Small
- removed C7: 3.3p, Capacitor_SMD:C_0805_2012Metric_Pad1.18x1.45mm_HandSolder, symbol Device:C_Small
- removed D1, D2: 4148, Diode_SMD:D_MicroMELF_Handsoldering, symbol Device:D_Small
- removed HS1001, HS1002: Heatsink, Heatsink:Heatsink_Aavid-TV5G_TO220_Horizontal, symbol Mechanical:Heatsink
- removed J1001: Conn_01x03, Connector_Molex:Molex_KK-254_AE-6410-03A_1x03_P2.54mm_Vertical, symbol Connector_Generic:Conn_01x03
- removed J1002, J1013: Conn_01x05, Connector_Molex:Molex_KK-254_AE-6410-05A_1x05_P2.54mm_Vertical, symbol Connector_Generic:Conn_01x05
- removed J1004: Conn_01x06, symbol Connector_Generic:Conn_01x06
- removed J1009, J1010, J1011, J1012: Conn_01x01, MountingHole:MountingHole_3.2mm_M3_Pad_Via, symbol Connector_Generic:Conn_01x01
- removed J2: Conn afficheur, Connector_Molex:Molex_KK-254_AE-6410-10A_1x10_P2.54mm_Vertical, symbol Connector_Generic:Conn_01x10
- removed J5: SMA, SMA_PINS:SMA_EDGE_NRW, symbol Connector:Conn_Coaxial
- removed J6: SMA, symbol Connector:Conn_Coaxial
- removed J7: BNC, symbol Connector:Conn_Coaxial
- removed Q1001: NTE2633, Package_TO_SOT_THT:TO-220-3_Horizontal_TabDown, symbol Device:Q_NPN_ECB
- removed Q1002: NTE2634, Package_TO_SOT_THT:TO-220-3_Horizontal_TabDown, symbol Device:Q_PNP_ECB
- removed R1001, R1002, R1003, R1004, R1005, R31, R32: 1k, Resistor_SMD:R_0603_1608Metric_Pad0.98x0.95mm_HandSolder, symbol Device:R_Small
- removed R26: 20k, Resistor_SMD:R_0603_1608Metric_Pad0.98x0.95mm_HandSolder, symbol Device:R_Small
- removed R27, R28: 680R, Resistor_SMD:R_0603_1608Metric_Pad0.98x0.95mm_HandSolder, symbol Device:R_Small
- removed R30: 27R, Resistor_SMD:R_0603_1608Metric_Pad0.98x0.95mm_HandSolder, symbol Device:R_Small
- removed R33, R34: 3R3, Resistor_SMD:R_1210_3225Metric_Pad1.30x2.65mm_HandSolder, symbol Device:R_Small
- removed R35: 47R, symbol Device:R_Small
- removed RV1: 100R, Potentiometer_THT:Potentiometer_Piher_PT-10-V10_Vertical_Hole, symbol Device:R_POT_TRIM
- removed SW1: Reset, symbol Switch:SW_Push
- removed SW3: Next, symbol Switch:SW_SPST
- removed SW4: Previous, symbol Switch:SW_SPST
- removed SW5: AC/DC, symbol Switch:SW_SPST
- removed SW6: 50R/Low Z, symbol Switch:SW_SPST
- removed U1: Pico, Pi_Pico:RPi_Pico_SMD_TH, symbol Pi_Pico:Pico
- removed U1001: L7812, Package_TO_SOT_SMD:TO-252-2, symbol Regulator_Linear:L7812
- removed U1002: L7912, Package_TO_SOT_SMD:TO-252-2, symbol Regulator_Linear:L7912
- removed U1003: L7805, Package_TO_SOT_SMD:TO-252-2, symbol Regulator_Linear:L7805
- removed U1004: L7905, Package_TO_SOT_SMD:TO-252-2, symbol Regulator_Linear:L7905
- removed U3: AD8055ARZ, Package_SO:SO-8_3.9x4.9mm_P1.27mm, symbol AD8055ARZ:AD8055ARZ
- added C1, C16, C28: 22u, Capacitor_SMD:C_1210_3225Metric, symbol Device:C_Small
- added C25: 100n, Capacitor_SMD:C_0603_1608Metric, symbol Device:C_Small
- added D4: 1N5819WS, Diode_SMD:D_SOD-323, symbol Device:D_Schottky_Small
- added H1, H2, H3, H4, H5, H6: MountingHole, MountingHole:MountingHole_3.2mm_M3, symbol Mechanical:MountingHole
- added J3: Conn_01x03, Connector_JST:JST_XH_S3B-XH-A_1x03_P2.50mm_Horizontal, symbol Connector_Generic:Conn_01x03
- added J4: BNC, Module:BNC_DOSIN_801_0050_Horizontal, symbol Connector:Conn_Coaxial
- added J5: Conn_01x14, Connector_PinSocket_2.54mm:PinSocket_1x14_P2.54mm_Vertical, symbol Connector_Generic:Conn_01x14
- added J9: Controls, Connector_PinSocket_2.54mm:PinSocket_1x06_P2.54mm_Vertical, symbol Connector_Generic:Conn_01x06
- added L7, L9: 47u, Inductor_SMD:L_Taiyo-Yuden_NR-50xx, symbol Device:L_Ferrite_Small
- added Q2: S9015, Package_TO_SOT_SMD:SOT-23, symbol Device:Q_PNP_BEC
- added R17, R18, R19: 27, Resistor_SMD:R_0603_1608Metric, symbol Device:R_Small
- added R43: 2k, Resistor_SMD:R_0603_1608Metric, symbol Device:R_Small
- added SW1: Prev, Module:Square_PB, symbol Switch:SW_DPDT_x2
- added SW2: Next, Module:Square_PB, symbol Switch:SW_DPDT_x2
- added U3: Pico, MCU_RaspberryPi_and_Boards:RPi_Pico_SMD, symbol MCU_RaspberryPi_and_Boards:Pico
- C3: value 100n -> 22u; footprint Capacitor_SMD:C_0805_2012Metric_Pad1.18x1.45mm_HandSolder -> Capacitor_SMD:C_1210_3225Metric; AVL1 (none) -> any/open; AVL2 (none) -> Samsung; AVL2 P/N (none) -> CL31A226KAHNNNE; LCSC (none) -> C12891
- J1: renamed from J1006; symbol Connector_Generic:Conn_01x01 -> Mechanical:MountingHole_Pad
- J2: renamed from J1007; symbol Connector_Generic:Conn_01x01 -> Mechanical:MountingHole_Pad
- J6: renamed from J1003; value Conn_01x06 -> Controls; footprint Connector_Molex:Molex_KK-254_AE-6410-06A_1x06_P2.54mm_Vertical -> Connector_PinHeader_2.54mm:PinHeader_1x06_P2.54mm_Vertical; AVL1 (none) -> any/open; AVL2 (none) -> XKB Connectivity; AVL2 P/N (none) -> X6511FV-06-C85D32; LCSC (none) -> C718239
- J7: renamed from J1008; symbol Connector_Generic:Conn_01x01 -> Mechanical:MountingHole_Pad
- J8: renamed from J1005; symbol Connector_Generic:Conn_01x01 -> Mechanical:MountingHole_Pad
- R1: renamed from R25; footprint Resistor_SMD:R_0603_1608Metric_Pad0.98x0.95mm_HandSolder -> Resistor_SMD:R_0603_1608Metric; AVL1 (none) -> any/open; LCSC (none) -> C319701
- R10: renamed from R11; footprint Resistor_SMD:R_0603_1608Metric_Pad0.98x0.95mm_HandSolder -> Resistor_SMD:R_0603_1608Metric; AVL1 (none) -> any/open; LCSC (none) -> C319701
- R11: renamed from R22; footprint Resistor_SMD:R_0603_1608Metric_Pad0.98x0.95mm_HandSolder -> Resistor_SMD:R_0603_1608Metric; AVL1 (none) -> any/open; LCSC (none) -> C309080
- R12: renamed from R10; footprint Resistor_SMD:R_0603_1608Metric_Pad0.98x0.95mm_HandSolder -> Resistor_SMD:R_0603_1608Metric; AVL1 (none) -> any/open; LCSC (none) -> C319701
- R13: renamed from R21; footprint Resistor_SMD:R_0603_1608Metric_Pad0.98x0.95mm_HandSolder -> Resistor_SMD:R_0603_1608Metric; AVL1 (none) -> any/open; LCSC (none) -> C309080
- R14: renamed from R9; footprint Resistor_SMD:R_0603_1608Metric_Pad0.98x0.95mm_HandSolder -> Resistor_SMD:R_0603_1608Metric; AVL1 (none) -> any/open; LCSC (none) -> C319701
- R15: renamed from R20; footprint Resistor_SMD:R_0603_1608Metric_Pad0.98x0.95mm_HandSolder -> Resistor_SMD:R_0603_1608Metric; AVL1 (none) -> any/open; LCSC (none) -> C309080
- R16: renamed from R8; footprint Resistor_SMD:R_0603_1608Metric_Pad0.98x0.95mm_HandSolder -> Resistor_SMD:R_0603_1608Metric; AVL1 (none) -> any/open; LCSC (none) -> C319701
- R2: renamed from R13; footprint Resistor_SMD:R_0603_1608Metric_Pad0.98x0.95mm_HandSolder -> Resistor_SMD:R_0603_1608Metric; AVL1 (none) -> any/open; LCSC (none) -> C319701
- R21: renamed from R19; footprint Resistor_SMD:R_0603_1608Metric_Pad0.98x0.95mm_HandSolder -> Resistor_SMD:R_0603_1608Metric; AVL1 (none) -> any/open; LCSC (none) -> C309080
- R22: renamed from R7; footprint Resistor_SMD:R_0603_1608Metric_Pad0.98x0.95mm_HandSolder -> Resistor_SMD:R_0603_1608Metric; AVL1 (none) -> any/open; LCSC (none) -> C319701
- R23: renamed from R18; footprint Resistor_SMD:R_0603_1608Metric_Pad0.98x0.95mm_HandSolder -> Resistor_SMD:R_0603_1608Metric; AVL1 (none) -> any/open; LCSC (none) -> C309080
- R24: renamed from R6; footprint Resistor_SMD:R_0603_1608Metric_Pad0.98x0.95mm_HandSolder -> Resistor_SMD:R_0603_1608Metric; AVL1 (none) -> any/open; LCSC (none) -> C319701
- R25: renamed from R17; footprint Resistor_SMD:R_0603_1608Metric_Pad0.98x0.95mm_HandSolder -> Resistor_SMD:R_0603_1608Metric; AVL1 (none) -> any/open; LCSC (none) -> C309080
- R26: renamed from R5; footprint Resistor_SMD:R_0603_1608Metric_Pad0.98x0.95mm_HandSolder -> Resistor_SMD:R_0603_1608Metric; AVL1 (none) -> any/open; LCSC (none) -> C319701
- R29: renamed from R16; footprint Resistor_SMD:R_0603_1608Metric_Pad0.98x0.95mm_HandSolder -> Resistor_SMD:R_0603_1608Metric; AVL1 (none) -> any/open; LCSC (none) -> C309080
- R3: renamed from R24; footprint Resistor_SMD:R_0603_1608Metric_Pad0.98x0.95mm_HandSolder -> Resistor_SMD:R_0603_1608Metric; AVL1 (none) -> any/open; LCSC (none) -> C309080
- R30: renamed from R4; footprint Resistor_SMD:R_0603_1608Metric_Pad0.98x0.95mm_HandSolder -> Resistor_SMD:R_0603_1608Metric; AVL1 (none) -> any/open; LCSC (none) -> C319701
- R4: renamed from R12; footprint Resistor_SMD:R_0603_1608Metric_Pad0.98x0.95mm_HandSolder -> Resistor_SMD:R_0603_1608Metric; AVL1 (none) -> any/open; LCSC (none) -> C319701
- R9: renamed from R23; footprint Resistor_SMD:R_0603_1608Metric_Pad0.98x0.95mm_HandSolder -> Resistor_SMD:R_0603_1608Metric; AVL1 (none) -> any/open; LCSC (none) -> C309080
- SW3: renamed from SW2; value Encodeur sur façade -> Encoder; footprint (none) -> Rotary_Encoder:RotaryEncoder_Alps_EC12E-Switch_Vertical_H20mm; AVL1 (none) -> Bourns Inc.; AVL1 P/N (none) -> PEC12R-4115F-S0012
Connections:
- net +5V is gone; now on net GND: C3.1
- net +3V3: now also C3.2, L9.1, U3.36 (3V3)
- net GND: now also SW3.C, SW3.S1, C1.1, C16.1, C25.1, C28.1, D4.2 (A), J3.2 (Pin_2), J4.2 (Ext), J5.2 (Pin_2), J9.6 (Pin_6), SW1.3 (C), SW2.2 (B), U3.13 (GND), U3.18 (GND), U3.23 (GND), U3.28 (GND), U3.3 (GND), U3.38 (GND), U3.42 (GND), U3.8 (GND); no longer C3.2
- net at R2.1: now also U3.1 (GPIO0)
- net at R24.1: now also U3.10 (GPIO7)
- net at R26.1: now also U3.11 (GPIO8)
- net at R30.1: now also U3.12 (GPIO9)
- net B_PR: now reaches J6.5 (Pin_5)
- net B_PR: now also J9.5 (Pin_5), SW1.2 (B), U3.15 (GPIO11)
- net B_NE: now reaches J6.4 (Pin_4)
- net B_NE: now also J9.4 (Pin_4), SW2.3 (C), U3.16 (GPIO12)
- net ENC_SW: now reaches J6.3 (Pin_3)
- net ENC_SW: now also SW3.S2, J9.3 (Pin_3), U3.17 (GPIO13)
- net ENC_B: now reaches J6.2 (Pin_2)
- net ENC_B: now also SW3.B, J9.2 (Pin_2), U3.19 (GPIO14)
- net at R4.1: now also U3.2 (GPIO1)
- net ENC_A: now reaches J6.1 (Pin_1)
- net ENC_A: now also SW3.A, J9.1 (Pin_1), U3.20 (GPIO15)
- net at R10.1: now also U3.4 (GPIO2)
- net at R12.1: now also U3.5 (GPIO3)
- net at R14.1: now also U3.6 (GPIO4)
- net at R16.1: now also U3.7 (GPIO5)
- net at R22.1: now also U3.9 (GPIO6)
- net amp/IN: now reaches R29.1, R30.2
- new net: R19.2, U3.25 (GPIO19)
- new net: R18.2, U3.26 (GPIO20)
- new net: R17.2, U3.29 (GPIO22)
- new net: Q2.1 (B), R43.2
- new net: D4.1 (K), L7.1, Q2.2 (E)
- new net +5VD: C1.2, U3.39 (VSYS)
- new net DAT/CMD: J5.5 (Pin_5), U3.22 (GPIO17)
- new net DC_PWM: U3.14 (GPIO10)
- new net LCD_3V3: C25.2, C28.2, J5.1 (Pin_1), J5.4 (Pin_4), L9.2, Q2.3 (C)
- new net LCD_CS: J5.3 (Pin_3), U3.21 (GPIO16)
- new net LCD_LED: C16.2, J5.8 (Pin_8), L7.2
- new net LCD_PWM: R43.1, U3.24 (GPIO18)
- new net MISO: J5.13 (Pin_13), J5.9 (Pin_9), R19.1
- new net MOSI: J5.12 (Pin_12), J5.6 (Pin_6), R17.1
- new net SCLK: J5.10 (Pin_10), J5.7 (Pin_7), R18.1
- new net TCH_CS: J5.11 (Pin_11), U3.27 (GPIO21)
- new net TCH_IRQ: J5.14 (Pin_14)
- new net amp/OUT: J4.1 (In)
- new net power/+12V_UNFIL: J3.1 (Pin_1)
- new net power/-12V_UNFIL: J3.3 (Pin_3)
- no-connect marks 14 -> 12
Other:
- added sheet amp (amp.kicad_sch)
- added sheet power (power.kicad_sch)
- note added: "30kHz+"
- note added: "P=100mW"
- note added: "P=165mW"
- note added: "P=33mW"
- note added: "XPT2046 touch"
- note removed: "+5V MISO CS Gnd SCK MOSI D/C Reset Led On Reset Raspi"
- note removed: "Inters, BNC et câble volants sur façade"
- note removed: "L7812CD2T-TR L7805ACD2T-TR L7905ACD2T-TR L7912CD2T-TR D²PAK (TO-263)"
- note removed: "To BNC and switches"
- note removed: "To encoder"
- note removed: "ajouter connecteur pour encodeur 5 fils connecteur next/previous 3 fils un fil blindé entre pcb et inters AC/CD-HI/LOW Z et sortie sur conn coax"
- note removed: "recommanded Primary power source RAC20-12DK or RAC20-15DK"
- note removed: "reglage I repos 25mA"
- moved on the sheet: J6, R1, R10, R11, R12, R13, R14, R15, R16, R2, R21, R22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
