File: amp.kicad_sch (KiCad schematic)
At the start: 36 parts, among them Q1 FZT653, Q3 FZT753, U4 LMH6658

Commit message: Make design more compact
Fitting it on a 100x70mm PCB means it's far cheaper to produce
Parts:
- renumbered C19 to C12, C17 to C14, C21 to C17, C23 to C19, C22 to C20, C13 to C21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
Connections:
- net IN renamed DAC_OUT
