File: awg.kicad_pcb (KiCad board)
At the start: 4 copper layers, 140 x 108.5 mm, 118 parts, among them J1 Conn_01x01, J2 Conn_01x01, J3 Conn_01x03, J4 BNC, J5 Conn_01x14, J6 Controls, J7 Conn_01x01, J8 Conn_01x01, J9 Controls, Q1 FZT653, Q2 S9015, Q3 FZT753, SW1 Prev, SW2 Next, SW3 Encoder, U1 BD9G101G, U2 BD9G101G, U3 Pico, U4 LMH6658

Commit message: Make design more compact
Fitting it on a 100x70mm PCB means it's far cheaper to produce
Parts:
- removed the H2 at (155.0, 65.0)
- removed H3, H5, H6: MountingHole, MountingHole:MountingHole_3.2mm_M3
- removed J9: Controls, Connector_PinSocket_2.54mm:PinSocket_1x06_P2.54mm_Vertical
- removed SW1: Prev, Module:Square_PB
- removed SW2: Next, Module:Square_PB
- removed SW3: Encoder, Rotary_Encoder:RotaryEncoder_Alps_EC12E-Switch_Vertical_H20mm
- J4: footprint Connector_Coaxial:BNC_TEConnectivity_1478035_Horizontal -> Module:BNC_DOSIN_801_0050_Horizontal
- L1: value 68u -> 47u; footprint Inductor_SMD:L_Wuerth_MAPI-3020 -> Inductor_SMD:L_Taiyo-Yuden_NR-50xx
- L2: renamed from L3; value 68u -> 47u; footprint Inductor_SMD:L_Wuerth_MAPI-3020 -> Inductor_SMD:L_Taiyo-Yuden_NR-50xx
- L3: renamed from L4; value 68u -> 47u; footprint Inductor_SMD:L_Wuerth_MAPI-3020 -> Inductor_SMD:L_Taiyo-Yuden_NR-50xx
- L4: renamed from L5; value 68u -> 47u; footprint Inductor_SMD:L_Wuerth_MAPI-3020 -> Inductor_SMD:L_Taiyo-Yuden_NR-50xx
- L5: renamed from L7; value 68u -> 47u; footprint Inductor_SMD:L_Wuerth_MAPI-3020 -> Inductor_SMD:L_Taiyo-Yuden_NR-50xx
- L6: renamed from L2; value 68u -> 47u; footprint Inductor_SMD:L_Wuerth_MAPI-3020 -> Inductor_SMD:L_Taiyo-Yuden_NR-50xx
- L8: renamed from L9; value 68u -> 47u; footprint Inductor_SMD:L_Wuerth_MAPI-3020 -> Inductor_SMD:L_Taiyo-Yuden_NR-50xx
- L9: renamed from L8; value 68u -> 47u; footprint Inductor_SMD:L_Wuerth_MAPI-3020 -> Inductor_SMD:L_Taiyo-Yuden_NR-50xx
- moved R19 141.9 mm to (133.1, 45.9)
- moved R18 141.8 mm to (94.7, 45.4)
- moved R21 141.8 mm to (94.7, 46.9)
- moved R24 141.8 mm to (94.7, 48.4)
- moved R27 141.8 mm to (94.7, 49.9)
- moved R22 141.8 mm to (133.1, 47.9)
- moved R25 141.8 mm to (133.1, 49.4)
- moved R17 141.4 mm to (91.7, 45.4)
- moved R20 141.4 mm to (91.7, 46.9)
- moved R23 141.4 mm to (91.7, 48.4)
- moved R26 141.4 mm to (91.7, 49.9)
- moved R28 141.4 mm to (91.7, 51.4), turned to 0 degrees
- moved D3 141.1 mm to (130.1, 55.9)
- moved TP3 141.0 mm to (84.1, 56.2)
- moved L8 140.6 mm to (130.6, 71.9)
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- renumbered C6 to C1, C3 to C10, C16 to C11, C19 to C12, C5 to C13, C17 to C14, C10 to C16, C21 to C17, C25 to C18, C23 to C19, C22 to C20, C13 to C21, C24 to C22, C14 to C23, C28 to C24, C20 to C25, C18 to C27, C27 to C28, C1 to C3, C11 to C4, C12 to C5, C9 to C6, C4 to C9, D4 to D3, D3 to D4, H4 to H2, J7 to J6, J8 to J7, J6 to J8, L6 to L7, Q2 to Q1, Q1 to Q2, R11 to R10, R12 to R11, R7 to R12, R21 to R17, R22 to R18, R17 to R19, R23 to R20, R24 to R21, R18 to R22, R25 to R23, R26 to R24, R19 to R25, R29 to R26, R30 to R27, R33 to R28, R36 to R29, R5 to R3, R35 to R30, R40 to R31, R39 to R32, R38 to R33, R41 to R34, R42 to R35, R43 to R36, R32 to R37, R20 to R38, R34 to R39, R3 to R4, R27 to R40, R31 to R41, R28 to R42, R37 to R43, R4 to R5, R9 to R7, R10 to R8, R8 to R9, TP5 to TP1, TP1 to TP2, TP2 to TP3, TP6 to TP5, TP3 to TP6, U2 to U1, U1 to U2
Connections:
- net /amp/IN renamed /amp/DAC_OUT
Routing:
- net /B_NE: track 185.1 -> 15.5 mm, vias 1 -> 0
- net /ENC_A: track 171.0 -> 15.0 mm, vias 2 -> 0
- net /ENC_B: track 158.9 -> 13.3 mm, vias 2 -> 0
- net /B_PR: track 140.9 -> 17.5 mm, vias 2 -> 0
- net /ENC_SW: track 138.3 -> 16.2 mm, vias 2 -> 0
- net -5V: track 55.0 -> 69.0 mm, vias 5 -> 3
- net Net-(C11-Pad2): track 9.03 -> 20.3 mm
- net -12V: track 34.4 -> 45.3 mm, vias 6 -> 7
- net /power/+12V_UNFIL: track 117.4 -> 127.5 mm, vias 3 -> 6
- net /power/-12V_UNFIL: track 152.2 -> 144.5 mm, vias 17 -> 15
- net GND: track 77.0 -> 70.1 mm, vias 142 -> 119
- net Net-(R15-Pad1): track 10.4 -> 3.59 mm
- net +5V: track 40.0 -> 46.2 mm, vias 6 -> 5
- net Net-(C18-Pad2): track 26.6 -> 32.5 mm
- net Net-(C21-Pad2): track 9.01 -> 3.40 mm
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- removed copper zone on F.Cu, net +12V
Other:
- board size 140 x 108.5 mm -> 100 x 75 mm
- board text added: "50Ω, ±3.3V"
