File: awg.kicad_sch (KiCad schematic)
At the start: 52 parts, among them J1 Conn_01x01, J2 Conn_01x01, J3 Conn_01x03, J4 BNC, J5 Conn_01x14, J6 Controls, J7 Conn_01x01, J8 Conn_01x01, J9 Controls, Q2 S9015, SW1 Prev, SW2 Next, SW3 Encoder, U3 Pico

Commit message: Make design more compact
Fitting it on a 100x70mm PCB means it's far cheaper to produce
Parts:
- removed H2, H3: MountingHole, MountingHole:MountingHole_3.2mm_M3, symbol Mechanical:MountingHole
- SW3: symbol Device:Rotary_Encoder_Switch -> Device:RotaryEncoder_Switch
- renumbered C3 to C10, C16 to C11, C25 to C18, C28 to C24, C1 to C3, D4 to D3, H4 to H2, J7 to J6, J8 to J7, J6 to J8, L7 to L5, L9 to L8, Q2 to Q1, R11 to R10, R12 to R11, R21 to R17, R22 to R18, R17 to R19, R23 to R20, R24 to R21, R18 to R22, R25 to R23, R26 to R24, R19 to R25, R29 to R26, R30 to R27, R43 to R36, R3 to R4, R4 to R5, R9 to R7, R10 to R8
Connections:
- net +3V3 renamed +3.3V
- net amp/IN renamed amp/DAC_OUT
- no-connect marks 12 -> 13
Other:
- sheet amp ports: added DAC_OUT; removed IN
- moved on the sheet: J8
